File: hardware/metering/ADE9153_With_Connector/ADE9153A_Ic.brd (EAGLE design)
At the start: 100 x 80 mm, 2 parts

Commit message: ADE9153Base
Parts:
- moved U$2 39.2 mm to (44.5, 55.9)
Routing:
- net 27: track 12.9 -> 8.96 mm
- net 29: track 12.0 -> 8.09 mm
- net 28: track 12.0 -> 8.14 mm
- net 26: track 13.7 -> 9.78 mm
- net 25: track 14.6 -> 10.7 mm
- net 30: track 12.8 -> 8.99 mm
- net 31: track 13.6 -> 9.80 mm
- net 32: track 14.4 -> 11.1 mm
- net 24: track 14.6 -> 12.6 mm
- net 23: track 13.7 -> 11.8 mm
- net 3: track 12.7 -> 10.9 mm
- net 22: track 12.7 -> 10.9 mm
- net 1: track 14.4 -> 12.7 mm
- net 2: track 13.6 -> 11.8 mm
- net 4: track 12.0 -> 10.4 mm
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