File: hardware/metering/ADE9153_With_Connector/ADE9153A_Ic.brd (EAGLE design)
At the start: 100 x 80 mm, 2 parts

Commit message: files change
Parts:
- removed U$2: ADE9153A_BASEADE9153A_BASE, ADE9153A_base:ADE9153A_BASE
- added J1, J2, J3, J4: (no value), con-amp:1X8MTA
- moved U$1 6.35 mm to (54.6, 38.1)
Connections:
- net 1: now also J2.8; no longer U$2.1
- net 10: now also J3.7; no longer U$2.10
- net 11: now also J3.6; no longer U$2.11
- net 12: now also J3.5; no longer U$2.12
- net 13: now also J3.4; no longer U$2.13
- net 14: now also J3.3; no longer U$2.14
- net 15: now also J3.2; no longer U$2.15
- net 16: now also J3.1; no longer U$2.16
- net 17: now also J4.8; no longer U$2.17
- net 18: now also J4.7; no longer U$2.18
- net 19: now also J4.6; no longer U$2.19
- net 2: now also J2.7; no longer U$2.2
- net 20: now also J4.5; no longer U$2.20
- net 21: now also J4.4; no longer U$2.21
- net 22: now also J4.3; no longer U$2.22
- net 23: now also J4.2; no longer U$2.23
- net 24: now also J4.1; no longer U$2.24
- net 25: now also J1.8; no longer U$2.25
- net 26: now also J1.7; no longer U$2.26
- net 27: now also J1.6; no longer U$2.27
- net 28: now also J1.5; no longer U$2.28
- net 29: now also J1.4; no longer U$2.29
- net 3: now also J2.6; no longer U$2.3
- net 30: now also J1.3; no longer U$2.30
- net 31: now also J1.2; no longer U$2.31
- net 32: now also J1.1; no longer U$2.32
- net 4: now also J2.5; no longer U$2.4
- net 5: now also J2.4; no longer U$2.5
- net 6: now also J2.3; no longer U$2.6
- net 7: now also J2.2; no longer U$2.7
- net 8: now also J2.1; no longer U$2.8
- net 9: now also J3.8; no longer U$2.9
Routing:
- net 9: track 14.4 -> 26.7 mm
- net 16: track 14.6 -> 26.8 mm
- net 10: track 13.7 -> 25.4 mm
- net 15: track 13.8 -> 25.2 mm
- net 8: track 14.4 -> 25.8 mm
- net 17: track 14.6 -> 25.9 mm
- net 14: track 12.7 -> 23.8 mm
- net 18: track 13.7 -> 24.5 mm
- net 7: track 13.7 -> 24.5 mm
- net 12: track 11.9 -> 22.6 mm
- net 11: track 12.9 -> 23.4 mm
- net 13: track 11.9 -> 22.3 mm
- net 1: track 14.4 -> 24.9 mm
- net 24: track 14.6 -> 24.9 mm
- net 19: track 12.8 -> 23.0 mm
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