File: hardware/metering/ADE9153_With_Connector/meetring ic.brd (EAGLE design)
At the start: 134.3 x 92.7 mm, 38 parts, among them J9 AK300/2-5,0-GRAU, Y1 12.288mhz

Commit message: ADE9153Base
Parts:
- added U$2: LIB1OPTION_HOLE, esp32_base_footprint:1X14MTA
Connections:
- net N$27: now also J1.1
Changed lines of the file:
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@@
 <attribute name="VALUE" x="84.04385" y="-26.223903125" size="1.27" layer="27" rot="R90"/>
 </element>
+<element name="U$2" library="esp32_base_footprint" package="1X14MTA" value="LIB1OPTION_HOLE" x="-14.1478" y="-20.1422" smashed="yes"/>
 </elements>
 <signals>
@@
 <wire x1="88.45865" y1="-24.768203125" x2="88.45865" y2="-27.11135" width="1.27" layer="1"/>
 <wire x1="88.45865" y1="-27.11135" x2="85.09" y2="-30.48" width="1.27" layer="1"/>
+<contactref element="J1" pad="1"/>
+<wire x1="88.45865" y1="-24.768203125" x2="88.45865" y2="-20.805803125" width="0" layer="19" extent="1-1"/>
 </signal>
 <signal name="GPIO19">
